Commit message: add gripper cob4-7

File: cob_hardware_config/robots/cob4-7/urdf/calibration_default.urdf.xacro (robot description, xacro)
@@ -63,4 +63,18 @@
 	<xacro:property name="def_arm_left_pitch" value="0"/>
 	<xacro:property name="def_arm_left_yaw" value="3.14159"/>
+    <!-- gripper right mount positions | relative to arm_right_7_link -->
+	<xacro:property name="def_gripper_right_x" value="0.0"/>
+	<xacro:property name="def_gripper_right_y" value="0.0"/>
+	<xacro:property name="def_gripper_right_z" value="0.0748"/>
+	<xacro:property name="def_gripper_right_roll" value="0.0"/>
+	<xacro:property name="def_gripper_right_pitch" value="0.0"/>
+	<xacro:property name="def_gripper_right_yaw" value="3.14159"/>
+	<!-- gripper left mount positions | relative to arm_left_7_link -->
+	<xacro:property name="def_gripper_left_x" value="0.0"/>
+	<xacro:property name="def_gripper_left_y" value="0.0"/>
+	<xacro:property name="def_gripper_left_z" value="0.0748"/>
+	<xacro:property name="def_gripper_left_roll" value="0.0"/>
+	<xacro:property name="def_gripper_left_pitch" value="0.0"/>
+	<xacro:property name="def_gripper_left_yaw" value="3.14159"/>
 	<!-- ***************************** -->
 	<!-- extrinsic camera calibration  -->

File: cob_hardware_config/robots/cob4-7/urdf/cob4-7.urdf.xacro (robot description, xacro)
@@ -67,4 +67,10 @@
     <origin xyz="${sensorring_x} ${sensorring_y} ${sensorring_z}" rpy="${sensorring_roll} ${sensorring_pitch} ${sensorring_yaw}" />
   </xacro:sensorring>
+  <xacro:gripper name="gripper_right" parent="arm_right_7_link">
+    <origin xyz="${gripper_right_x} ${gripper_right_y} ${gripper_right_z}" rpy="${gripper_right_roll} ${gripper_right_pitch} ${gripper_right_yaw}" />
+  </xacro:gripper>
+  <xacro:gripper name="gripper_left" parent="arm_left_7_link">
+    <origin xyz="${gripper_left_x} ${gripper_left_y} ${gripper_left_z}" rpy="${gripper_left_roll} ${gripper_left_pitch} ${gripper_left_yaw}" />
+  </xacro:gripper>
    <!-- Mojin Robotics set up with kinect camera in sensorring part (not true for Cob4-7)-->
   <!--xacro:cob_kinect_v0 name="sensorring_cam3d" ros_topic="sensorring_cam3d" parent="sensorring_link" update_rate="30" data_skip="9">

File: cob_hardware_config/robots/cob4-7/urdf/properties.urdf.xacro (robot description, xacro)
@@ -66,4 +66,18 @@
 	<xacro:property name="arm_left_pitch" value="${def_arm_left_pitch+offset_arm_left_pitch}"/>
 	<xacro:property name="arm_left_yaw" value="${def_arm_left_yaw+offset_arm_left_yaw}"/>
+    <!-- gripper mount positions | relative to arm_7_link -->
+	<xacro:property name="gripper_right_x" value="${def_gripper_right_x+offset_gripper_right_x}"/>
+	<xacro:property name="gripper_right_y" value="${def_gripper_right_y+offset_gripper_right_y}"/>
+	<xacro:property name="gripper_right_z" value="${def_gripper_right_z+offset_gripper_right_z}"/>
+	<xacro:property name="gripper_right_roll" value="${def_gripper_right_roll+offset_gripper_right_roll}"/>
+	<xacro:property name="gripper_right_pitch" value="${def_gripper_right_pitch+offset_gripper_right_pitch}"/>
+	<xacro:property name="gripper_right_yaw" value="${def_gripper_right_yaw+offset_gripper_right_yaw}"/>
+	<!-- gripper mount positions | relative to arm_7_link -->
+	<xacro:property name="gripper_left_x" value="${def_gripper_left_x+offset_gripper_left_x}"/>
+	<xacro:property name="gripper_left_y" value="${def_gripper_left_y+offset_gripper_left_y}"/>
+	<xacro:property name="gripper_left_z" value="${def_gripper_left_z+offset_gripper_left_z}"/>
+	<xacro:property name="gripper_left_roll" value="${def_gripper_left_roll+offset_gripper_left_roll}"/>
+	<xacro:property name="gripper_left_pitch" value="${def_gripper_left_pitch+offset_gripper_left_pitch}"/>
+	<xacro:property name="gripper_left_yaw" value="${def_gripper_left_yaw+offset_gripper_left_yaw}"/>
 	<!-- *********************************** -->
 	<!-- kinematic chain reference positions -->
